File: FxT-65_Circuit.kicad_sch (KiCad schematic)
At the start: 0 parts

Commit message: マザボ回路を追加
Parts:
- added C1: 30pF, symbol Device:C
- added C2, C3, C5, C6: 0.1u, symbol Device:C
- added C4: 50p, symbol Device:C
- added C7: 10u, symbol FxT-65-Mother-rescue:CP1-Device
- added D1, D?: DIODE, symbol pspice:DIODE
- added D2, D3: LED, symbol Device:LED
- added J1: BUS_conn, symbol Connector_Generic:Conn_01x40
- added J10, J12: SD_socket_conn, symbol Connector_Generic:Conn_01x07
- added J11, J13: Conn_01x02, symbol Connector_Generic:Conn_01x02
- added J14: AKI_SD_Card_Slot, symbol FxT-65-Mother-rescue:AKI_SD_Card_Slot-ponzu840w
- added J15: POW_PINS, symbol Connector_Generic:Conn_02x05_Odd_Even
- added J2: Mini-DIN-6, symbol Connector:Mini-DIN-6
- added J6: Clocks_Out, symbol Connector_Generic:Conn_02x05_Odd_Even
- added J7: UART_Socket, symbol Connector_Generic:Conn_01x06
- added J8: PS/2_conn, symbol Connector_Generic:Conn_01x02
- added J9: USB_B_Micro, symbol Connector:USB_B_Micro
- added JP1: Clock_Sel, symbol FxT-65-Mother-rescue:Jumper_NC_Small-Device
- added JP2, JP3, JP4: Jumper_NC_Small, symbol FxT-65-Mother-rescue:Jumper_NC_Small-Device
- added R10: 1M, symbol Device:R
- added R11, R12, R13, R6, R8, R9, R?: 1.2k, symbol Device:R
- added R14, R15, R16, R3, R4, R5: 1.5k, symbol Device:R
- added R17: 4.6k, symbol Device:R
- added R? (x2): 1k, symbol Device:R
- added SW1: BUT_NMI, symbol Switch:SW_Push
- added SW2: BUT_RES, symbol Switch:SW_Push
- added SW3: POW, symbol Switch:SW_DIP_x01
- added U1: 74125, symbol 74xx_IEEE:74125
- added U10: 74LS191, symbol 74xx:74LS191
- added U11: CY62256-70PC, Package_DIP:DIP-28_W15.24mm, symbol Memory_RAM:CY62256-70PC
- added U12: HN58V66AFP-10, symbol FxT-65-Mother-rescue:HN58V66AFP-10-ponzu840w
- added U2: 7400, symbol 74xx:7400
- added U3: WD65C22, symbol FxT-65-Mother-rescue:WD65C22-65xx
- added U4: 74LVC244, symbol 74xx:74HC244
- added U5, U6: 74LS138, symbol 74xx:74LS138
- added U7: WD65C02, symbol FxT-65-Mother-rescue:WD65C02-65xx
- added U8: KHO-HC1-TS, symbol FxT-65-Mother-rescue:KHO-HC1-TS-ponzu840w
- added U9: W65C51N, symbol FxT-65-Mother-rescue:W65C51N-65xx
- added U?: TCM809, symbol Power_Supervisor:TCM809
- added Y1: Crystal, symbol Device:Crystal
Connections:
- new net: R8.1, U7.2 (RDY)
- new net: U2.1, U2.2, U3.22 (R/~{W}), U7.34 (R/~{W}), U9.28 (R/~{W})
- new net: R12.2, U7.36 (BE)
- new net: R11.2, U7.38 (~{SO})
- new net: C2.1, J11.1 (Pin_1), R?.1, SW1.2, U7.6 (~{NMI})
- new net: R9.1, U7.7 (SYNC)
- new net: R16.2, U9.10 (Tx_Data)
- new net: R15.2, U9.12 (Rx_Data)
- new net: U6.15 (O0), U9.3 (~{CS1})
- new net: C1.1, R10.2, U9.6 (XTLI), Y1.1
- new net: R10.1, U9.7 (XLT0), Y1.2
- new net: R14.2, U9.8 (~{RTS})
- new net: R?.2, U3.14 (PB4)
- new net: R?.2, U3.15 (PB5)
- new net: U3.16 (PB6), U4.6 (1A2)
- new net: U1.1 (EN), U2.10, U2.9, U3.17 (PB7)
- new net: U3.18 (CB1), U4.2 (1A0)
- new net: U1.2 (D), U1.6 (O), U3.19 (CB2)
- new net: D1.2 (A), U3.21 (~{IRQ})
- new net: U3.23 (~{CS2}), U6.14 (O1)
- new net: U12.20 (/CE), U5.7 (O7)
- new net: U5.9 (O6), U6.5 (E2)
- new net: D3.2 (A), R17.1
- new net: J2.1, J8.2 (Pin_2)
- new net: J2.5, J8.1 (Pin_1)
- new net: U2.3, U2.4
- new net: J7.2 (Pin_2), R14.1
- new net: J7.4 (Pin_4), R15.1
- new net: J7.5 (Pin_5), R16.1
- new net: J10.4 (Pin_4), U4.14 (1Y2)
- new net: J10.5 (Pin_5), R4.1, U4.16 (1Y1)
- new net: J10.6 (Pin_6), R3.1, U4.18 (1Y0)
- new net: J10.3 (Pin_3), R3.2, R4.2, U4.20 (VCC)
- new net: U1.3 (O), U4.4 (1A1)
- new net: U1.4 (EN), U2.8
- new net: J10.7 (Pin_7), U1.5 (D)
- new net: D2.1 (K), J12.3 (Pin_3), J14.2 (VDD/3.3VOUT)
- new net: D2.2 (A), R5.2
- new net: J12.4 (Pin_4), J14.4 (D3/CS), R5.1
- new net: J6.5 (Pin_5), J6.6 (Pin_6), JP2.1, U10.2 (Q1)
- new net: J6.3 (Pin_3), J6.4 (Pin_4), JP1.1, U10.3 (Q0)
- new net: J6.7 (Pin_7), J6.8 (Pin_8), JP3.1, U10.6 (Q2)
- new net: J6.10 (Pin_10), J6.9 (Pin_9), JP4.1, U10.7 (Q3)
- new net: J12.2 (Pin_2), J14.1 (GND)
- new net: J12.1 (Pin_1), J14.12 (5Vin)
- new net: J12.5 (Pin_5), J14.5 (CMD/MOSI)
- new net: J12.6 (Pin_6), J14.6 (CLK)
- new net: J12.7 (Pin_7), J14.7 (D0/MISO)
- new net: J9.1 (VBUS), SW3.2
- new net: D?.2 (A), U?.2 (~{RESET})
- new net 16MHz: C4.1, J1.31 (Pin_31), J6.1 (Pin_1), J6.2 (Pin_2), U10.14 (Cp), U8.5 (Out)
- new net 60Hz: J1.32 (Pin_32), U3.39 (CA2)
- new net A0: J1.15 (Pin_15), U11.10 (A0), U12.10 (A0), U3.38 (RS0), U7.9 (A0), U9.13 (RS0)
- new net A1: J1.16 (Pin_16), U11.9 (A1), U12.9 (A1), U3.37 (RS1), U7.10 (A1), U9.14 (RS1)
- new net A10: J1.25 (Pin_25), U11.21 (A10), U12.21 (A10), U6.2 (A1), U7.19 (A10)
- new net A11: J1.26 (Pin_26), U11.23 (A11), U12.23 (A11), U6.3 (A2), U7.20 (A11)
- new net A12: J1.27 (Pin_27), U11.2 (A12), U12.2 (A12), U5.1 (A0), U7.22 (A12)
- new net A13: J1.28 (Pin_28), U11.26 (A13), U5.2 (A1), U7.23 (A13)
- new net A14: U11.1 (A14), U5.3 (A2), U7.24 (A14)
- new net A15: U11.20 (~{CS}), U5.6 (E3), U7.25 (A15)
- new net A2: J1.17 (Pin_17), U11.8 (A2), U12.8 (A2), U3.36 (RS2), U7.11 (A2)
- new net A3: J1.18 (Pin_18), U11.7 (A3), U12.7 (A3), U3.35 (RS3), U7.12 (A3)
- new net A4: J1.19 (Pin_19), U11.6 (A4), U12.6 (A4), U7.13 (A4)
- new net A5: J1.20 (Pin_20), U11.5 (A5), U12.5 (A5), U7.14 (A5)
- new net A6: J1.21 (Pin_21), U11.4 (A6), U12.4 (A6), U7.15 (A6)
- new net A7: J1.22 (Pin_22), U11.3 (A7), U12.3 (A7), U7.16 (A7)
- new net A8: J1.23 (Pin_23), U11.25 (A8), U12.25 (A8), U7.17 (A8)
- new net A9: J1.24 (Pin_24), U11.24 (A9), U12.24 (A9), U6.1 (A0), U7.18 (A9)
- new net CRTC_CS: J1.30 (Pin_30), U6.12 (O3)
- new net D0: J1.7 (Pin_7), U11.11 (Q0), U12.11 (I/O0), U3.33 (D0), U7.33 (D0), U9.18 (D0)
- new net D1: J1.8 (Pin_8), U11.12 (Q1), U12.12 (I/O1), U3.32 (D1), U7.32 (D1), U9.19 (D1)
- new net D2: J1.9 (Pin_9), U11.13 (Q2), U12.13 (I/O2), U3.31 (D2), U7.31 (D2), U9.20 (D2)
- new net D3: J1.10 (Pin_10), U11.15 (Q3), U12.15 (I/O3), U3.30 (D3), U7.30 (D3), U9.21 (D3)
- new net D4: J1.11 (Pin_11), U11.16 (Q4), U12.16 (I/O4), U3.29 (D4), U7.29 (D4), U9.22 (D4)
- new net D5: J1.12 (Pin_12), U11.17 (Q5), U12.17 (I/O5), U3.28 (D5), U7.28 (D5), U9.23 (D5)
- new net D6: J1.13 (Pin_13), U11.18 (Q6), U12.18 (I/O6), U3.27 (D6), U7.27 (D6), U9.24 (D6)
- new net D7: J1.14 (Pin_14), U11.19 (Q7), U12.19 (I/O7), U3.26 (D7), U7.26 (D7), U9.25 (D7)
- new net GND: C1.2, C2.2, C3.1, C4.2, C5.1, C5.2, C6.1, C6.2, C7.1, C7.2, D3.1 (K), J1.1 (Pin_1), J1.2 (Pin_2), J10.1 (Pin_1), J10.2 (Pin_2), J11.2 (Pin_2), J13.1 (Pin_1), J15.1 (Pin_1), J15.10 (Pin_10), J15.2 (Pin_2), J15.3 (Pin_3), J15.4 (Pin_4), J15.5 (Pin_5), J15.6 (Pin_6), J15.7 (Pin_7), J15.8 (Pin_8), J15.9 (Pin_9), J2.3, J2.4, J7.1 (Pin_1), J9.5 (GND), R11.1, R12.1, R13.2, R17.2, R6.1, R8.2, R9.2, R?.2, SW1.1, SW2.2, SW3.1, U1.10 (EN), U1.12 (D), U1.13 (EN), U1.14 (VCC), U1.14 (VCC), U1.14 (VCC), U1.14 (VCC), U1.7 (GND), U1.7 (GND), U1.7 (GND), U1.7 (GND), U1.9 (D), U10.1 (P1), U10.10 (P2), U10.11 (Pl), U10.15 (P0), U10.16 (VCC), U10.4 (Ce), U10.5 (D/U), U10.8 (GND), U10.9 (P3), U11.14 (GND), U11.22 (~{OE}), U11.28 (VCC), U12.14 (Vss), U12.22 (/OE), U12.26 (/RES), U12.27 (/WE), U12.28 (Vcc), U3.1 (GND), U3.20 (VCC), U3.24 (CS1), U4.1 (1OE), U4.10 (GND), U4.11 (2A3), U4.13 (2A2), U4.15 (2A1), U4.17 (2A0), U4.19 (2OE), U4.8 (1A3), U5.16 (VCC), U5.4 (E1), U5.5 (E2), U5.8 (GND), U6.16 (VCC), U6.4 (E1), U6.6 (E3), U6.8 (GND), U7.21 (GND), U7.8 (VCC), U8.4 (GND), U8.8 (5V), U9.1 (GND), U9.15 (VCC), U9.16 (~{DCD}), U9.17 (~{DSR}), U9.2 (CS0), U?.1 (GND), U?.3 (VCC)
- new net IRQ: D1.1 (K), J1.5 (Pin_5), R6.2, U7.4 (~{IRQ}), U9.26 (~{IRQ})
- new net PAD_CLK: U3.12 (PB2)
- new net PAD_DAT: U3.10 (PB0)
- new net PAD_PTS: U3.11 (PB1)
- new net PS2_CLK: R?.1
- new net PS2_DAT: R?.1
- new net RES: C3.2, D?.1 (K), J1.4 (Pin_4), J13.2 (Pin_2), R13.1, SW2.1, U3.34 (~{RESET}), U7.40 (~{RESET}), U9.4 (~{RESET})
- new net WE: J1.6 (Pin_6), U11.27 (~{WE}), U2.6
- new net YMZ_CS: J1.29 (Pin_29), U6.13 (O2)
- new net φ2: J1.3 (Pin_3), JP1.2, JP2.2, JP3.2, JP4.2, U2.5, U3.25 (PHI2), U7.37 (PHI2), U9.27 (PHI2)
- no-connect marks 0 -> 58
Other:
- note added: "1MHz"
- note added: "2MHz"
- note added: "3.3V"
- note added: "4MHz"
- note added: "5V"
- note added: "8MHz"
- note added: "CLK"
- note added: "CMD=MOSI"
- note added: "D0=MISO"
- note added: "D3=CS"
- note added: "DAT"
- note added: "GND"
- note added: "RTS"
- note added: "RX"
- note added: "TX"
- note added: "VCC"
- note added: "clk"
- note added: "cs"
- note added: "cs0"
- note added: "data i/o"
- note added: "i/o sel"
- note added: "miso"
- note added: "mosi"
- note added: "xN"
- note added: "φ2"

Commit message: 全ボードを追加
Parts:
- removed C1: 30pF, symbol Device:C
- removed C2, C3, C5, C6: 0.1u, symbol Device:C
- removed C4: 50p, symbol Device:C
- removed C7: 10u, symbol FxT-65-Mother-rescue:CP1-Device
- removed D1, D?: DIODE, symbol pspice:DIODE
- removed D2, D3: LED, symbol Device:LED
- removed J1: BUS_conn, symbol Connector_Generic:Conn_01x40
- removed J10, J12: SD_socket_conn, symbol Connector_Generic:Conn_01x07
- removed J11, J13: Conn_01x02, symbol Connector_Generic:Conn_01x02
- removed J14: AKI_SD_Card_Slot, symbol FxT-65-Mother-rescue:AKI_SD_Card_Slot-ponzu840w
- removed J15: POW_PINS, symbol Connector_Generic:Conn_02x05_Odd_Even
- removed J2: Mini-DIN-6, symbol Connector:Mini-DIN-6
- removed J6: Clocks_Out, symbol Connector_Generic:Conn_02x05_Odd_Even
- removed J7: UART_Socket, symbol Connector_Generic:Conn_01x06
- removed J8: PS/2_conn, symbol Connector_Generic:Conn_01x02
- removed J9: USB_B_Micro, symbol Connector:USB_B_Micro
- removed JP1: Clock_Sel, symbol FxT-65-Mother-rescue:Jumper_NC_Small-Device
- removed JP2, JP3, JP4: Jumper_NC_Small, symbol FxT-65-Mother-rescue:Jumper_NC_Small-Device
- removed R10: 1M, symbol Device:R
- removed R11, R12, R13, R6, R8, R9, R?: 1.2k, symbol Device:R
- removed R14, R15, R16, R3, R4, R5: 1.5k, symbol Device:R
- removed R17: 4.6k, symbol Device:R
- removed R? (x2): 1k, symbol Device:R
- removed SW1: BUT_NMI, symbol Switch:SW_Push
- removed SW2: BUT_RES, symbol Switch:SW_Push
- removed SW3: POW, symbol Switch:SW_DIP_x01
- removed U1: 74125, symbol 74xx_IEEE:74125
- removed U10: 74LS191, symbol 74xx:74LS191
- removed U11: CY62256-70PC, Package_DIP:DIP-28_W15.24mm, symbol Memory_RAM:CY62256-70PC
- removed U12: HN58V66AFP-10, symbol FxT-65-Mother-rescue:HN58V66AFP-10-ponzu840w
- removed U2: 7400, symbol 74xx:7400
- removed U3: WD65C22, symbol FxT-65-Mother-rescue:WD65C22-65xx
- removed U4: 74LVC244, symbol 74xx:74HC244
- removed U5, U6: 74LS138, symbol 74xx:74LS138
- removed U7: WD65C02, symbol FxT-65-Mother-rescue:WD65C02-65xx
- removed U8: KHO-HC1-TS, symbol FxT-65-Mother-rescue:KHO-HC1-TS-ponzu840w
- removed U9: W65C51N, symbol FxT-65-Mother-rescue:W65C51N-65xx
- removed U?: TCM809, symbol Power_Supervisor:TCM809
- removed Y1: Crystal, symbol Device:Crystal
Connections:
- no-connect marks 58 -> 0
Other:
- added sheet chiina-dazzler (chiina-dazzler.kicad_sch)
- added sheet mother (mother.kicad_sch)
- added sheet psg (psg.kicad_sch)
- added sheet tiny-psg (tiny-psg.kicad_sch)
- note added: "1ch サブ・サウンドボード"
- note added: "サウンドボード"
- note added: "ビデオボード"
- note added: "マザーボード"
- note removed: "1MHz"
- note removed: "2MHz"
- note removed: "3.3V"
- note removed: "4MHz"
- note removed: "5V"
- note removed: "8MHz"
- note removed: "CLK"
- note removed: "CMD=MOSI"
- note removed: "D0=MISO"
- note removed: "D3=CS"
- note removed: "DAT"
- note removed: "GND"
- note removed: "RTS"
- note removed: "RX"
- note removed: "TX"
- note removed: "VCC"
- note removed: "clk"
- note removed: "cs"
- note removed: "cs0"
- note removed: "data i/o"
- note removed: "i/o sel"
- note removed: "miso"
- note removed: "mosi"
- note removed: "xN"
- note removed: "φ2"

Commit message: aaa
Parts:
- added C10, C12, C14, C8: 0.1u, symbol Device:C
- added C11: 50p, symbol Device:C
- added C13: 10u, symbol FxT-65-Mother-rescue:CP1-Device
- added C9: 30pF, symbol Device:C
- added D4, D6: DIODE, symbol pspice:DIODE
- added D5, D7: LED, symbol Device:LED
- added J16, J18: SD_socket_conn, symbol Connector_Generic:Conn_01x07
- added J17, J19: Conn_01x02, symbol Connector_Generic:Conn_01x02
- added J20: AKI_SD_Card_Slot, symbol FxT-65-Mother-rescue:AKI_SD_Card_Slot-ponzu840w
- added J21: Clocks_Out, symbol Connector_Generic:Conn_02x05_Odd_Even
- added J22: UART_Socket, symbol Connector_Generic:Conn_01x06
- added J23: POW_PINS, symbol Connector_Generic:Conn_02x05_Odd_Even
- added J24: USB_B_Micro, symbol Connector:USB_B_Micro
- added J3: BUS_conn, symbol Connector_Generic:Conn_01x40
- added J4: PS/2_conn, symbol Connector_Generic:Conn_01x02
- added J5: Mini-DIN-6, symbol Connector:Mini-DIN-6
- added JP5: Clock_Sel, symbol FxT-65-Mother-rescue:Jumper_NC_Small-Device
- added JP6, JP7, JP8: Jumper_NC_Small, symbol FxT-65-Mother-rescue:Jumper_NC_Small-Device
- added R1, R2: 1k, symbol Device:R
- added R18, R27, R28, R29, R30, R7: 1.5k, symbol Device:R
- added R19, R20, R21, R22, R24, R25, R26: 1.2k, symbol Device:R
- added R23: 1M, symbol Device:R
- added R31: 4.6k, symbol Device:R
- added SW4: BUT_NMI, symbol Switch:SW_Push
- added SW5: BUT_RES, symbol Switch:SW_Push
- added SW6: POW, symbol Switch:SW_DIP_x01
- added U13: 74125, symbol 74xx_IEEE:74125
- added U14: 7400, symbol 74xx:7400
- added U15: WD65C22, symbol FxT-65-Mother-rescue:WD65C22-65xx
- added U16: 74LVC244, symbol 74xx:74HC244
- added U17, U18: 74LS138, symbol 74xx:74LS138
- added U19: WD65C02, symbol FxT-65-Mother-rescue:WD65C02-65xx
- added U20: KHO-HC1-TS, symbol FxT-65-Mother-rescue:KHO-HC1-TS-ponzu840w
- added U21: TCM809, symbol Power_Supervisor:TCM809
- added U22: W65C51N, symbol FxT-65-Mother-rescue:W65C51N-65xx
- added U23: 74LS191, symbol 74xx:74LS191
- added U24: CY62256-70PC, Package_DIP:DIP-28_W15.24mm, symbol Memory_RAM:CY62256-70PC
- added U25: HN58V66AFP-10, symbol FxT-65-Mother-rescue:HN58V66AFP-10-ponzu840w
- added Y2: Crystal, symbol Device:Crystal
Connections:
- new net: R1.2, U15.14 (PB4)
- new net: J21.5 (Pin_5), J21.6 (Pin_6), JP6.1, U23.2 (Q1)
- new net: J21.3 (Pin_3), J21.4 (Pin_4), JP5.1, U23.3 (Q0)
- new net: J21.7 (Pin_7), J21.8 (Pin_8), JP7.1, U23.6 (Q2)
- new net: J21.10 (Pin_10), J21.9 (Pin_9), JP8.1, U23.7 (Q3)
- new net: D7.2 (A), R31.1
- new net: C8.1, J17.1 (Pin_1), R22.1, SW4.2, U19.6 (~{NMI})
- new net: J16.4 (Pin_4), U16.14 (1Y2)
- new net: J16.5 (Pin_5), R18.1, U16.16 (1Y1)
- new net: J16.6 (Pin_6), R7.1, U16.18 (1Y0)
- new net: U15.18 (CB1), U16.2 (1A0)
- new net: J16.3 (Pin_3), R18.2, R7.2, U16.20 (VCC)
- new net: U13.3 (O), U16.4 (1A1)
- new net: U15.16 (PB6), U16.6 (1A2)
- new net: R2.2, U15.15 (PB5)
- new net: D5.1 (K), J18.3 (Pin_3), J20.2 (VDD/3.3VOUT)
- new net: D5.2 (A), R27.2
- new net: J18.1 (Pin_1), J20.12 (5Vin)
- new net: J18.2 (Pin_2), J20.1 (GND)
- new net: J18.4 (Pin_4), J20.4 (D3/CS), R27.1
- new net: J18.5 (Pin_5), J20.5 (CMD/MOSI)
- new net: J18.6 (Pin_6), J20.6 (CLK)
- new net: J18.7 (Pin_7), J20.7 (D0/MISO)
- new net: J22.5 (Pin_5), R30.1
- new net: R30.2, U22.10 (Tx_Data)
- new net: R19.1, U19.2 (RDY)
- new net: U14.1, U14.2, U15.22 (R/~{W}), U19.34 (R/~{W}), U22.28 (R/~{W})
- new net: R26.2, U19.36 (BE)
- new net: R25.2, U19.38 (~{SO})
- new net: R21.1, U19.7 (SYNC)
- new net: D6.2 (A), U21.2 (~{RESET})
- new net: U13.1 (EN), U14.10, U14.9, U15.17 (PB7)
- new net: U13.2 (D), U13.6 (O), U15.19 (CB2)
- new net: D4.2 (A), U15.21 (~{IRQ})
- new net: U15.23 (~{CS2}), U18.14 (O1)
- new net: J24.1 (VBUS), SW6.2
- new net: C9.1, R23.2, U22.6 (XTLI), Y2.1
- new net: U17.7 (O7), U25.20 (/CE)
- new net: U17.9 (O6), U18.5 (E2)
- new net: J22.2 (Pin_2), R28.1
- new net: J22.4 (Pin_4), R29.1
- new net: R29.2, U22.12 (Rx_Data)
- new net: U18.15 (O0), U22.3 (~{CS1})
- new net: R23.1, U22.7 (XLT0), Y2.2
- new net: R28.2, U22.8 (~{RTS})
- new net: J16.7 (Pin_7), U13.5 (D)
- new net: J4.1 (Pin_1), J5.5
- new net: J4.2 (Pin_2), J5.1
- new net: U13.4 (EN), U14.8
- new net: U14.3, U14.4
- new net 16MHz: C11.1, J21.1 (Pin_1), J21.2 (Pin_2), J3.31 (Pin_31), U20.5 (Out), U23.14 (Cp)
- new net 60Hz: J3.32 (Pin_32), U15.39 (CA2)
- new net A0: J3.15 (Pin_15), U15.38 (RS0), U19.9 (A0), U22.13 (RS0), U24.10 (A0), U25.10 (A0)
- new net A1: J3.16 (Pin_16), U15.37 (RS1), U19.10 (A1), U22.14 (RS1), U24.9 (A1), U25.9 (A1)
- new net A10: J3.25 (Pin_25), U18.2 (A1), U19.19 (A10), U24.21 (A10), U25.21 (A10)
- new net A11: J3.26 (Pin_26), U18.3 (A2), U19.20 (A11), U24.23 (A11), U25.23 (A11)
- new net A12: J3.27 (Pin_27), U17.1 (A0), U19.22 (A12), U24.2 (A12), U25.2 (A12)
- new net A13: J3.28 (Pin_28), U17.2 (A1), U19.23 (A13), U24.26 (A13)
- new net A14: U17.3 (A2), U19.24 (A14), U24.1 (A14)
- new net A15: U17.6 (E3), U19.25 (A15), U24.20 (~{CS})
- new net A2: J3.17 (Pin_17), U15.36 (RS2), U19.11 (A2), U24.8 (A2), U25.8 (A2)
- new net A3: J3.18 (Pin_18), U15.35 (RS3), U19.12 (A3), U24.7 (A3), U25.7 (A3)
- new net A4: J3.19 (Pin_19), U19.13 (A4), U24.6 (A4), U25.6 (A4)
- new net A5: J3.20 (Pin_20), U19.14 (A5), U24.5 (A5), U25.5 (A5)
- new net A6: J3.21 (Pin_21), U19.15 (A6), U24.4 (A6), U25.4 (A6)
- new net A7: J3.22 (Pin_22), U19.16 (A7), U24.3 (A7), U25.3 (A7)
- new net A8: J3.23 (Pin_23), U19.17 (A8), U24.25 (A8), U25.25 (A8)
- new net A9: J3.24 (Pin_24), U18.1 (A0), U19.18 (A9), U24.24 (A9), U25.24 (A9)
- new net CRTC_CS: J3.30 (Pin_30), U18.12 (O3)
- new net D0: J3.7 (Pin_7), U15.33 (D0), U19.33 (D0), U22.18 (D0), U24.11 (Q0), U25.11 (I/O0)
- new net D1: J3.8 (Pin_8), U15.32 (D1), U19.32 (D1), U22.19 (D1), U24.12 (Q1), U25.12 (I/O1)
- new net D2: J3.9 (Pin_9), U15.31 (D2), U19.31 (D2), U22.20 (D2), U24.13 (Q2), U25.13 (I/O2)
- new net D3: J3.10 (Pin_10), U15.30 (D3), U19.30 (D3), U22.21 (D3), U24.15 (Q3), U25.15 (I/O3)
- new net D4: J3.11 (Pin_11), U15.29 (D4), U19.29 (D4), U22.22 (D4), U24.16 (Q4), U25.16 (I/O4)
- new net D5: J3.12 (Pin_12), U15.28 (D5), U19.28 (D5), U22.23 (D5), U24.17 (Q5), U25.17 (I/O5)
- new net D6: J3.13 (Pin_13), U15.27 (D6), U19.27 (D6), U22.24 (D6), U24.18 (Q6), U25.18 (I/O6)
- new net D7: J3.14 (Pin_14), U15.26 (D7), U19.26 (D7), U22.25 (D7), U24.19 (Q7), U25.19 (I/O7)
- new net GND: C10.1, C11.2, C12.1, C12.2, C13.1, C13.2, C14.1, C14.2, C8.2, C9.2, D7.1 (K), J16.1 (Pin_1), J16.2 (Pin_2), J17.2 (Pin_2), J19.1 (Pin_1), J22.1 (Pin_1), J23.1 (Pin_1), J23.10 (Pin_10), J23.2 (Pin_2), J23.3 (Pin_3), J23.4 (Pin_4), J23.5 (Pin_5), J23.6 (Pin_6), J23.7 (Pin_7), J23.8 (Pin_8), J23.9 (Pin_9), J24.5 (GND), J3.1 (Pin_1), J3.2 (Pin_2), J5.3, J5.4, R19.2, R20.1, R21.2, R22.2, R24.2, R25.1, R26.1, R31.2, SW4.1, SW5.2, SW6.1, U13.10 (EN), U13.12 (D), U13.13 (EN), U13.14 (VCC), U13.14 (VCC), U13.14 (VCC), U13.14 (VCC), U13.7 (GND), U13.7 (GND), U13.7 (GND), U13.7 (GND), U13.9 (D), U15.1 (GND), U15.20 (VCC), U15.24 (CS1), U16.1 (1OE), U16.10 (GND), U16.11 (2A3), U16.13 (2A2), U16.15 (2A1), U16.17 (2A0), U16.19 (2OE), U16.8 (1A3), U17.16 (VCC), U17.4 (E1), U17.5 (E2), U17.8 (GND), U18.16 (VCC), U18.4 (E1), U18.6 (E3), U18.8 (GND), U19.21 (GND), U19.8 (VCC), U20.4 (GND), U20.8 (5V), U21.1 (GND), U21.3 (VCC), U22.1 (GND), U22.15 (VCC), U22.16 (~{DCD}), U22.17 (~{DSR}), U22.2 (CS0), U23.1 (P1), U23.10 (P2), U23.11 (Pl), U23.15 (P0), U23.16 (VCC), U23.4 (Ce), U23.5 (D/U), U23.8 (GND), U23.9 (P3), U24.14 (GND), U24.22 (~{OE}), U24.28 (VCC), U25.14 (Vss), U25.22 (/OE), U25.26 (/RES), U25.27 (/WE), U25.28 (Vcc)
- new net IRQ: D4.1 (K), J3.5 (Pin_5), R20.2, U19.4 (~{IRQ}), U22.26 (~{IRQ})
- new net PAD_CLK: U15.12 (PB2)
- new net PAD_DAT: U15.10 (PB0)
- new net PAD_PTS: U15.11 (PB1)
- new net PS2_CLK: R2.1
- new net PS2_DAT: R1.1
- new net RES: C10.2, D6.1 (K), J19.2 (Pin_2), J3.4 (Pin_4), R24.1, SW5.1, U15.34 (~{RESET}), U19.40 (~{RESET}), U22.4 (~{RESET})
- new net WE: J3.6 (Pin_6), U14.6, U24.27 (~{WE})
- new net YMZ_CS: J3.29 (Pin_29), U18.13 (O2)
- new net φ2: J3.3 (Pin_3), JP5.2, JP6.2, JP7.2, JP8.2, U14.5, U15.25 (PHI2), U19.37 (PHI2), U22.27 (PHI2)
- no-connect marks 0 -> 58
Other:
- removed sheet chiina-dazzler
- removed sheet mother
- removed sheet psg
- removed sheet tiny-psg
- note added: "1MHz"
- note added: "2MHz"
- note added: "3.3V"
- note added: "4MHz"
- note added: "5V"
- note added: "8MHz"
- note added: "CLK"
- note added: "CMD=MOSI"
- note added: "D0=MISO"
- note added: "D3=CS"
- note added: "DAT"
- note added: "GND"
- note added: "RTS"
- note added: "RX"
- note added: "TX"
- note added: "VCC"
- note added: "clk"
- note added: "cs"
- note added: "cs0"
- note added: "data i/o"
- note added: "i/o sel"
- note added: "miso"
- note added: "mosi"
- note added: "xN"
- note added: "φ2"
- note removed: "1ch サブ・サウンドボード"
- note removed: "サウンドボード"
- note removed: "ビデオボード"
- note removed: "マザーボード"
